Commit message: refactor(ros): remove MPU6050 dependency from active robot stack

File: Raspberrypi/catkin_ws/src/clbrobot_project/clbrobot/urdf/cleanscout_geometry.xacro (robot description, xacro)
@@ -9,7 +9,4 @@
   <xacro:property name="wheel_radius" value="0.04" />
   <xacro:property name="wheel_thickness" value="0.03" />
-  <xacro:property name="imu_length" value="0.02" />
-  <xacro:property name="imu_width" value="0.015" />
-  <xacro:property name="imu_height" value="0.001" />
   <xacro:property name="laser_radius" value="0.04" />
   <xacro:property name="laser_height" value="0.04" />
@@ -46,19 +43,4 @@
     <origin xyz="0.0745 0.0065 0.592" rpy="0 0 0" />
   </joint>
-  <link name="imu_link">
-    <visual>
-      <geometry>
-        <box size="${imu_length} ${imu_width} ${imu_height}" />
-      </geometry>
-      <material name="green">
-        <color rgba="0.2 0.8 0.3 1.0" />
-      </material>
-    </visual>
-  </link>
-  <joint name="base_link_to_imu_joint" type="fixed">
-    <parent link="base_link" />
-    <child link="imu_link" />
-    <origin xyz="0.093 0.072 0.0725" rpy="0 0 0" />
-  </joint>
   <xacro:macro name="wheel_link" params="name x y">
     <link name="${name}">

Commit message: feat(ros): establish C-4.1.8 rear blind safety baseline

File: Raspberrypi/catkin_ws/src/clbrobot_project/clbrobot/urdf/cleanscout_geometry.xacro (robot description, xacro)
@@ -1,8 +1,8 @@
 <?xml version="1.0"?>
 <robot xmlns:xacro="http://www.ros.org/wiki/xacro" name="cleanscout">
-  <!-- Base geometry uses the current navigation convention:
-       base_link is the center of the four-wheel rectangle. -->
-  <xacro:property name="base_length" value="0.353" />
-  <xacro:property name="base_width" value="0.217" />
+  <!-- New body outline measured on 2026-07-20. Until an offset is measured,
+       navigation treats base_link as the geometric center of this box. -->
+  <xacro:property name="base_length" value="0.244" />
+  <xacro:property name="base_width" value="0.255" />
   <xacro:property name="base_height" value="0.024" />
   <xacro:property name="wheel_diameter" value="0.08" />
@@ -13,5 +13,5 @@
   <link name="base_link">
     <visual>
-      <origin xyz="0.0415 0 ${base_height / 2.0}" rpy="0 0 0" />
+      <origin xyz="0 0 ${base_height / 2.0}" rpy="0 0 0" />
       <geometry>
         <box size="${base_length} ${base_width} ${base_height}" />
@@ -22,5 +22,5 @@
     </visual>
     <collision>
-      <origin xyz="0.0415 0 ${base_height / 2.0}" rpy="0 0 0" />
+      <origin xyz="0 0 ${base_height / 2.0}" rpy="0 0 0" />
       <geometry>
         <box size="${base_length} ${base_width} ${base_height}" />
